File: hardware_old/ADM3260_Breakout.kicad_sch (KiCad schematic)
At the start: 21 parts, among them J11 CONN_05LOCK_LONGPADS, J22 BNCPTH, Q1 BSS84, Q2 BSH105, Q3 BSS84, U22 Atlas Scientific OEM, U4 ADM3260ARSZ

Commit message: schematic done, board needs replication for all 4 channels
Parts:
- renumbered U4 to U1
