File: hardware-new/BREAD_Slice.kicad_pcb (KiCad board)
At the start: 4 copper layers, 100.1 x 144.9 mm, 181 parts, among them J1 Conn_01x10_Female, J2 Conn_Coaxial, J3 Conn_Coaxial, J4 Conn_Coaxial, J5 Conn_Coaxial, J6 Conn_Coaxial, J7 Conn_Coaxial, J8 Conn_Coaxial, J9 Conn_Coaxial, Q1 BSS84, Q10 BSS84, Q11 BS170, Q12 BSS84, Q2 BS170, Q3 BSS84, Q4 BSS84, Q5 BS170, Q6 BSS84, Q7 BSS84, Q8 BS170, Q9 BSS84, U1 AP63205, U2 Atlas Scientific OEM, U3 ADM3260ARSZ, U4 ADM3260ARSZ, U5 Atlas Scientific OEM, U6 Atlas Scientific OEM, U7 ADM3260ARSZ, U8 Atlas Scientific OEM, U9 ADM3260ARSZ

Commit message: finalized pcb
Parts:
- removed the C13 at (116.0, 68.3)
- removed the C13 at (116.0, 156.5)
- removed the C13 at (115.9, 126.9)
- removed the C13 at (115.9, 97.7)
- removed the C14 at (115.9, 94.1)
- removed the C14 at (116.0, 152.9)
- removed the C14 at (115.9, 64.7)
- removed the C14 at (115.9, 123.3)
- removed the C15 at (115.8, 66.5)
- removed the C15 at (115.8, 154.7)
- removed the C15 at (115.7, 95.9)
- removed the C15 at (115.8, 125.1)
- removed the C16 at (115.8, 92.3)
- removed the C16 at (115.8, 151.1)
- removed the C16 at (115.8, 62.9)
- removed the C16 at (115.8, 121.5)
- removed the C17 at (128.2, 69.5)
- removed the C17 at (128.1, 98.9)
- removed the C17 at (128.2, 128.1)
- removed the C17 at (128.2, 157.7)
- removed the C18 at (131.0, 152.1)
- removed the C18 at (130.9, 63.9)
- removed the C18 at (130.9, 93.3)
- removed the C18 at (130.9, 122.5)
- removed the C19 at (126.4, 69.4)
- removed the C19 at (126.4, 157.5)
- removed the C19 at (126.3, 98.7)
- removed the C19 at (126.4, 127.9)
- removed the C20 at (129.1, 152.2)
- removed the C20 at (129.1, 122.6)
- removed the C20 at (129.0, 93.4)
- removed the C20 at (129.1, 64.0)
- removed the J2 at (153.1, 100.3)
- removed the J2 at (153.1, 70.9)
- removed the J2 at (153.1, 129.5)
- removed the J3 at (153.1, 116.6)
- removed the J3 at (153.1, 58.0)
- removed the J3 at (153.1, 87.4)
- removed JP10 (x2), JP11 (x2), JP12 (x2), JP7, JP8, JP9 (x4): SolderJumper_3_Open, Jumper:SolderJumper-3_P1.3mm_Open_RoundedPad1.0x1.5mm
- removed Logo1: Logo_Open_Hardware_Small, Symbol:OSHW-Symbol_6.7x6mm_SilkScreen
- removed the Q4 at (111.3, 102.7)
- removed the Q4 at (111.3, 131.9)
- removed the Q4 at (111.4, 161.5)
- removed the Q4 at (111.4, 73.3)
- removed the Q5 at (111.3, 99.1)
- removed the Q5 at (111.3, 128.3)
- removed the Q5 at (111.4, 157.9)
- removed the Q5 at (111.3, 69.7)
- removed the Q6 at (115.3, 131.9)
- removed the Q6 at (115.4, 161.5)
- removed the Q6 at (115.3, 73.3)
- removed the Q6 at (115.3, 102.7)
- removed the R10 at (128.9, 66.7)
- removed the R10 at (128.9, 154.9)
- removed the R10 at (128.8, 96.1)
- removed the R10 at (128.9, 125.3)
- removed the R11 at (133.5, 122.2)
- removed the R11 at (133.5, 151.8)
- removed the R11 at (133.5, 63.6)
- removed the R11 at (133.4, 93.0)
- removed the R12 at (133.4, 89.6)
- removed the R12 at (133.5, 118.8)
- removed the R12 at (133.5, 60.3)
- removed the R12 at (133.5, 148.4)
- removed the R7 at (112.7, 88.6)
- removed the R7 at (112.7, 59.2)
- removed the R7 at (112.8, 147.4)
- removed the R7 at (112.7, 117.8)
- removed the R8 at (112.7, 121.2)
- removed the R8 at (112.7, 92.0)
- removed the R8 at (112.7, 62.6)
- removed the R8 at (112.8, 150.8)
- removed the R9 at (131.4, 126.2)
- removed the R9 at (131.4, 155.8)
- removed the R9 at (131.4, 67.7)
- removed the R9 at (131.3, 97.0)
- removed the U2 at (146.7, 99.8)
- removed the U2 at (146.7, 70.4)
- removed the U2 at (146.7, 129.0)
- removed the U3 at (92.6, 112.3)
- removed the U4 at (122.4, 93.4)
- removed the U4 at (122.5, 64.0)
- removed the U4 at (122.4, 122.6)
- removed the U4 at (122.5, 152.2)
- added C13: 0.1u, Capacitor_SMD:C_0603_1608Metric_Pad1.08x0.95mm_HandSolder, F.Cu at (115.8, 122.9)
- added C14: 0.1u, Capacitor_SMD:C_0603_1608Metric_Pad1.08x0.95mm_HandSolder, F.Cu at (115.9, 126.6)
- added C15: 10u, Capacitor_SMD:C_0805_2012Metric_Pad1.18x1.45mm_HandSolder, F.Cu at (115.7, 121.1)
- added C16: 10u, Capacitor_SMD:C_0805_2012Metric_Pad1.18x1.45mm_HandSolder, F.Cu at (115.7, 124.7)
- added C17: 10u, Capacitor_SMD:C_0805_2012Metric_Pad1.18x1.45mm_HandSolder, F.Cu at (128.8, 127.7)
- added C18: 0.1u, Capacitor_SMD:C_0603_1608Metric_Pad1.08x0.95mm_HandSolder, F.Cu at (127.0, 127.6)
- added C19: 0.1u, Capacitor_SMD:C_0603_1608Metric_Pad1.08x0.95mm_HandSolder, F.Cu at (130.8, 122.1)
- added C20: 10u, Capacitor_SMD:C_0805_2012Metric_Pad1.18x1.45mm_HandSolder, F.Cu at (129.0, 122.3)
- added G***: LOGO, kml-custom:FAST-Logo-XXXLarge, F.Cu at (85.9, 72.6)
- added Q4: BSS84, Package_TO_SOT_SMD:SOT-23, F.Cu at (111.3, 131.5)
- added Q5: BS170, Package_TO_SOT_SMD:SOT-23, F.Cu at (111.2, 127.9)
- added Q6: BSS84, Package_TO_SOT_SMD:SOT-23, F.Cu at (115.2, 131.5)
- added R10: 10k, Resistor_SMD:R_0603_1608Metric_Pad0.98x0.95mm_HandSolder, F.Cu at (128.8, 125.0)
- added R11: 4.7k, Resistor_SMD:R_0603_1608Metric_Pad0.98x0.95mm_HandSolder, F.Cu at (133.4, 121.8)
- added R12: 4.7k, Resistor_SMD:R_0603_1608Metric_Pad0.98x0.95mm_HandSolder, F.Cu at (133.4, 118.5)
- added R7: 4.7k, Resistor_SMD:R_0603_1608Metric_Pad0.98x0.95mm_HandSolder, F.Cu at (112.6, 117.4)
- added R8: 4.7k, Resistor_SMD:R_0603_1608Metric_Pad0.98x0.95mm_HandSolder, F.Cu at (112.6, 120.8)
- added R9: 16.2k, Resistor_SMD:R_0603_1608Metric_Pad0.98x0.95mm_HandSolder, F.Cu at (131.3, 125.9)
- added REF**: OSHW-Symbol_8.9x8mm_SilkScreen, Symbol:OSHW-Symbol_8.9x8mm_SilkScreen, F.Cu at (71.6, 147.9)
- added U2: ADM3260ARSZ, kml-custom:RS_20_ADI-L, F.Cu at (122.4, 152.9)
- added U4: ADM3260ARSZ, kml-custom:RS_20_ADI-L, F.Cu at (122.3, 122.3)
- JP3, JP4, JP5, JP6: moved to B.Cu
- U6, U8: value Atlas Scientific OEM -> ADM3260ARSZ; footprint kml-custom:Atlas_OEM -> kml-custom:RS_20_ADI-L
- U7, U9: value ADM3260ARSZ -> Atlas Scientific OEM; footprint kml-custom:RS_20_ADI-L -> kml-custom:Atlas_OEM
- moved JP3 131.2 mm to (145.7, 156.7), turned to 180 degrees
- moved JP6 123.2 mm to (145.8, 66.6), turned to 180 degrees
- moved JP5 120.0 mm to (145.7, 96.0), turned to 180 degrees
- moved JP4 117.7 mm to (145.7, 126.0), turned to 180 degrees
- moved JP2 89.1 mm to (101.1, 159.4), turned to 180 degrees
- moved JP1 88.1 mm to (98.2, 156.8), turned to 180 degrees
- moved U6 86.9 mm to (122.4, 92.3)
- moved U8 86.4 mm to (122.4, 62.8)
- moved U5 63.2 mm to (146.6, 128.7), turned to 90 degrees
- moved R3 62.7 mm to (131.3, 156.5), turned to 90 degrees
- moved R5 58.6 mm to (133.4, 152.5), turned to 90 degrees
- moved R4 58.5 mm to (128.8, 155.6)
- moved U7 55.6 mm to (146.6, 98.7), turned to 90 degrees
- moved R6 55.5 mm to (133.4, 149.2), turned to -90 degrees
- moved U9 55.4 mm to (146.7, 69.2), turned to 90 degrees
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- renumbered U2 to U3
Connections:
- net /Isolated Atlas OEM Module/PROBE_IN1 renamed /Isolated Atlas OEM Module1/SIG_1
- net /Isolated Atlas OEM Module/PROBE_IN4 renamed /Isolated Atlas OEM Module1/REF_2
- net /Isolated Atlas OEM Module1/ADM3260 I2C Isolator1/VSEL renamed /ADM3260 I2C Isolator1/VSEL
- net /Isolated Atlas OEM Module1/PROBE_IN1 renamed /Isolated Atlas OEM Module2/SIG_1
- net /Isolated Atlas OEM Module1/PROBE_IN4 renamed /Isolated Atlas OEM Module2/REF_2
- A1 pad 10: /SCL_SOFT -> /SDA_SOFT
- A1 pad 11: /EN1 -> /EN4
- A1 pad 12: /EN2 -> /EN3
- A1 pad 13: /EN3 -> /EN2
- A1 pad 14: /EN4 -> /EN1
- A1 pad 9: /SDA_SOFT -> /SCL_SOFT
- C10 pad 1: /Isolated Atlas OEM Module1/ISO_GND -> /ISO1_GND
- C10 pad 2: /Isolated Atlas OEM Module1/ISO_3V3 -> /ISO1_3V3
- C11 pad 1: /Isolated Atlas OEM Module1/ISO_GND -> /ISO1_GND
- C11 pad 2: /Isolated Atlas OEM Module1/ISO_3V3 -> /ISO1_3V3
- C12 pad 1: /Isolated Atlas OEM Module1/ISO_GND -> /ISO1_GND
- C12 pad 2: /Isolated Atlas OEM Module1/ISO_3V3 -> /ISO1_3V3
- C21 pad 2: /Isolated Atlas OEM Module2/ADM3260 I2C Isolator1/AVCC -> /ADM3260 I2C Isolator3/AVCC
- C22 pad 2: /Isolated Atlas OEM Module2/ADM3260 I2C Isolator1/AVCC -> /ADM3260 I2C Isolator3/AVCC
- C23 pad 2: /Isolated Atlas OEM Module2/ADM3260 I2C Isolator1/AVCC -> /ADM3260 I2C Isolator3/AVCC
- C24 pad 2: /Isolated Atlas OEM Module2/ADM3260 I2C Isolator1/AVCC -> /ADM3260 I2C Isolator3/AVCC
- C25 pad 1: /Isolated Atlas OEM Module2/ISO_GND -> /ISO3_GND
- C25 pad 2: /Isolated Atlas OEM Module2/ISO_3V3 -> /ISO3_3V3
- C26 pad 1: /Isolated Atlas OEM Module2/ISO_GND -> /ISO3_GND
- C26 pad 2: /Isolated Atlas OEM Module2/ISO_3V3 -> /ISO3_3V3
- C27 pad 1: /Isolated Atlas OEM Module2/ISO_GND -> /ISO3_GND
- C27 pad 2: /Isolated Atlas OEM Module2/ISO_3V3 -> /ISO3_3V3
- C28 pad 1: /Isolated Atlas OEM Module2/ISO_GND -> /ISO3_GND
- C28 pad 2: /Isolated Atlas OEM Module2/ISO_3V3 -> /ISO3_3V3
- C29 pad 2: /Isolated Atlas OEM Module3/ADM3260 I2C Isolator1/AVCC -> /ADM3260 I2C Isolator4/AVCC
- C30 pad 2: /Isolated Atlas OEM Module3/ADM3260 I2C Isolator1/AVCC -> /ADM3260 I2C Isolator4/AVCC
- C31 pad 2: /Isolated Atlas OEM Module3/ADM3260 I2C Isolator1/AVCC -> /ADM3260 I2C Isolator4/AVCC
- C32 pad 2: /Isolated Atlas OEM Module3/ADM3260 I2C Isolator1/AVCC -> /ADM3260 I2C Isolator4/AVCC
- C33 pad 1: /Isolated Atlas OEM Module3/ISO_GND -> /ISO4_GND
- C33 pad 2: /Isolated Atlas OEM Module3/ISO_3V3 -> /ISO4_3V3
- C34 pad 1: /Isolated Atlas OEM Module3/ISO_GND -> /ISO4_GND
- C34 pad 2: /Isolated Atlas OEM Module3/ISO_3V3 -> /ISO4_3V3
- C35 pad 1: /Isolated Atlas OEM Module3/ISO_GND -> /ISO4_GND
- C35 pad 2: /Isolated Atlas OEM Module3/ISO_3V3 -> /ISO4_3V3
- C36 pad 1: /Isolated Atlas OEM Module3/ISO_GND -> /ISO4_GND
- C36 pad 2: /Isolated Atlas OEM Module3/ISO_3V3 -> /ISO4_3V3
- C5 pad 2: /Isolated Atlas OEM Module1/ADM3260 I2C Isolator1/AVCC -> /ADM3260 I2C Isolator1/AVCC
- C6 pad 2: /Isolated Atlas OEM Module1/ADM3260 I2C Isolator1/AVCC -> /ADM3260 I2C Isolator1/AVCC
- C7 pad 2: /Isolated Atlas OEM Module1/ADM3260 I2C Isolator1/AVCC -> /ADM3260 I2C Isolator1/AVCC
- C8 pad 2: /Isolated Atlas OEM Module1/ADM3260 I2C Isolator1/AVCC -> /ADM3260 I2C Isolator1/AVCC
- C9 pad 1: /Isolated Atlas OEM Module1/ISO_GND -> /ISO1_GND
- C9 pad 2: /Isolated Atlas OEM Module1/ISO_3V3 -> /ISO1_3V3
- J2 pad 2: /Isolated Atlas OEM Module/REF_1 -> /Isolated Atlas OEM Module1/REF_1
- J3 pad 1: /Isolated Atlas OEM Module/PROBE_IN3 -> /Isolated Atlas OEM Module1/SIG_2
- J4 pad 2: /Isolated Atlas OEM Module1/REF_1 -> /Isolated Atlas OEM Module2/REF_1
- J5 pad 1: /Isolated Atlas OEM Module1/PROBE_IN3 -> /Isolated Atlas OEM Module2/SIG_2
- J6 pad 1: /Isolated Atlas OEM Module2/PROBE_IN1 -> /Isolated Atlas OEM Module3/SIG_1
- J6 pad 2: /Isolated Atlas OEM Module2/REF_1 -> /Isolated Atlas OEM Module3/REF_1
- J7 pad 1: /Isolated Atlas OEM Module2/PROBE_IN3 -> /Isolated Atlas OEM Module3/SIG_2
- J7 pad 2: /Isolated Atlas OEM Module2/PROBE_IN4 -> /Isolated Atlas OEM Module3/REF_2
- J8 pad 1: /Isolated Atlas OEM Module3/PROBE_IN1 -> /Isolated Atlas OEM Module4/SIG_1
- J8 pad 2: /Isolated Atlas OEM Module3/REF_1 -> /Isolated Atlas OEM Module4/REF_1
- J9 pad 1: /Isolated Atlas OEM Module3/PROBE_IN3 -> /Isolated Atlas OEM Module4/SIG_2
- J9 pad 2: /Isolated Atlas OEM Module3/PROBE_IN4 -> /Isolated Atlas OEM Module4/REF_2
- JP1 pad 1: /SCL1_5V -> /SCL_SOFT
- JP1 pad 2: /SCL_SOFT -> /SCL_5V
- JP2 pad 1: /SDA1_5V -> /SDA_SOFT
- JP2 pad 2: /SDA_SOFT -> /SDA_5V
- JP3 pad 1: /SCL2_5V -> /Isolated Atlas OEM Module1/SIG_2
- JP3 pad 2: /SCL_SOFT -> /Isolated Atlas OEM Module1/PRB_IN2_SEL
- JP3 pad 3: /I2C_CLK -> /Isolated Atlas OEM Module1/REF_1
- JP4 pad 1: /SDA2_5V -> /Isolated Atlas OEM Module2/SIG_2
- JP4 pad 2: /SDA_SOFT -> /Isolated Atlas OEM Module2/PRB_IN2_SEL
- JP4 pad 3: /I2C_DAT -> /Isolated Atlas OEM Module2/REF_1
- JP5 pad 1: /SCL3_5V -> /Isolated Atlas OEM Module3/SIG_2
- JP5 pad 2: /SCL_SOFT -> /Isolated Atlas OEM Module3/PRB_IN2_SEL
- JP5 pad 3: /I2C_CLK -> /Isolated Atlas OEM Module3/REF_1
- JP6 pad 1: /SDA3_5V -> /Isolated Atlas OEM Module4/SIG_2
- JP6 pad 2: /SDA_SOFT -> /Isolated Atlas OEM Module4/PRB_IN2_SEL
- JP6 pad 3: /I2C_DAT -> /Isolated Atlas OEM Module4/REF_1
- Q1 pad 1: /EN2 -> /EN1
- Q12 pad 2: /Isolated Atlas OEM Module3/ADM3260 I2C Isolator1/AVCC -> /ADM3260 I2C Isolator4/AVCC
- Q2 pad 2: /EN2 -> /EN1
- Q3 pad 2: /Isolated Atlas OEM Module1/ADM3260 I2C Isolator1/AVCC -> /ADM3260 I2C Isolator1/AVCC
- Q9 pad 2: /Isolated Atlas OEM Module2/ADM3260 I2C Isolator1/AVCC -> /ADM3260 I2C Isolator3/AVCC
- R1 pad 1: /Isolated Atlas OEM Module1/ADM3260 I2C Isolator1/AVCC -> +5V
- R1 pad 2: /SCL2_5V -> /SCL_5V
- R13 pad 1: /Isolated Atlas OEM Module2/ADM3260 I2C Isolator1/AVCC -> +5V
- R13 pad 2: /SCL3_5V -> /SCL_5V
- R14 pad 1: /Isolated Atlas OEM Module2/ADM3260 I2C Isolator1/AVCC -> +5V
- R14 pad 2: /SDA3_5V -> /SDA_5V
- R15 pad 1: /Isolated Atlas OEM Module2/ISO_3V3 -> /ISO3_3V3
- R15 pad 2: /Isolated Atlas OEM Module2/ADM3260 I2C Isolator1/VSEL -> /ADM3260 I2C Isolator3/VSEL
- R16 pad 1: /Isolated Atlas OEM Module2/ADM3260 I2C Isolator1/VSEL -> /ADM3260 I2C Isolator3/VSEL
- R16 pad 2: /Isolated Atlas OEM Module2/ISO_GND -> /ISO3_GND
- R17 pad 1: /Isolated Atlas OEM Module2/ISO_3V3 -> /ISO3_3V3
- R17 pad 2: /Isolated Atlas OEM Module2/SDA_3V3 -> /SDA3_3V3
- R18 pad 1: /Isolated Atlas OEM Module2/ISO_3V3 -> /ISO3_3V3
- R18 pad 2: /Isolated Atlas OEM Module2/SCL_3V3 -> /SCL3_3V3
- R19 pad 1: /Isolated Atlas OEM Module3/ADM3260 I2C Isolator1/AVCC -> +5V
- R19 pad 2: /SCL4_5V -> /SCL_5V
- R2 pad 1: /Isolated Atlas OEM Module1/ADM3260 I2C Isolator1/AVCC -> +5V
- R2 pad 2: /SDA2_5V -> /SDA_5V
- R20 pad 1: /Isolated Atlas OEM Module3/ADM3260 I2C Isolator1/AVCC -> +5V
- R20 pad 2: /SDA4_5V -> /SDA_5V
- R21 pad 1: /Isolated Atlas OEM Module3/ISO_3V3 -> /ISO4_3V3
- R21 pad 2: /Isolated Atlas OEM Module3/ADM3260 I2C Isolator1/VSEL -> /ADM3260 I2C Isolator4/VSEL
- R22 pad 1: /Isolated Atlas OEM Module3/ADM3260 I2C Isolator1/VSEL -> /ADM3260 I2C Isolator4/VSEL
- R22 pad 2: /Isolated Atlas OEM Module3/ISO_GND -> /ISO4_GND
- R23 pad 1: /Isolated Atlas OEM Module3/ISO_3V3 -> /ISO4_3V3
- R23 pad 2: /Isolated Atlas OEM Module3/SDA_3V3 -> /SDA4_3V3
- R24 pad 1: /Isolated Atlas OEM Module3/ISO_3V3 -> /ISO4_3V3
- R24 pad 2: /Isolated Atlas OEM Module3/SCL_3V3 -> /SCL4_3V3
- R3 pad 1: /Isolated Atlas OEM Module1/ISO_3V3 -> /ISO1_3V3
- R4 pad 2: /Isolated Atlas OEM Module1/ISO_GND -> /ISO1_GND
- R5 pad 1: /Isolated Atlas OEM Module1/ISO_3V3 -> /ISO1_3V3
- R5 pad 2: /Isolated Atlas OEM Module1/SDA_3V3 -> /SDA1_3V3
- R6 pad 1: /Isolated Atlas OEM Module1/ISO_3V3 -> /ISO1_3V3
- R6 pad 2: /Isolated Atlas OEM Module1/SCL_3V3 -> /SCL1_3V3
- U3 pad P1: /Isolated Atlas OEM Module/SDA_3V3 -> /SDA1_3V3
- U3 pad P10: /Isolated Atlas OEM Module/SCL_3V3 -> /SCL1_3V3
- U3 pad P3: /Isolated Atlas OEM Module/ISO_3V3 -> /ISO1_3V3
- U3 pad P5: /Isolated Atlas OEM Module/PROBE_IN2 -> /Isolated Atlas OEM Module1/PRB_IN2_SEL
- U3 pad P6: /Isolated Atlas OEM Module/PROBE_IN3 -> /Isolated Atlas OEM Module1/SIG_2
- U3 pad P8: /Isolated Atlas OEM Module/ISO_GND -> /ISO1_GND
- U5 pad P1: /Isolated Atlas OEM Module1/SDA_3V3 -> /SDA2_3V3
- U5 pad P10: /Isolated Atlas OEM Module1/SCL_3V3 -> /SCL2_3V3
- U5 pad P3: /Isolated Atlas OEM Module1/ISO_3V3 -> /ISO2_3V3
- U5 pad P5: /Isolated Atlas OEM Module1/PROBE_IN2 -> /Isolated Atlas OEM Module2/PRB_IN2_SEL
- U5 pad P6: /Isolated Atlas OEM Module1/PROBE_IN3 -> /Isolated Atlas OEM Module2/SIG_2
- U5 pad P8: /Isolated Atlas OEM Module1/ISO_GND -> /ISO2_GND
Routing:
- net /SCL_5V: track 0.00 -> 186.5 mm
- net /SDA_5V: track 0.00 -> 178.6 mm, vias 0 -> 6
- net /INT4: track 0.00 -> 146.5 mm, vias 0 -> 1
- net /EN4: track 0.00 -> 124.5 mm, vias 0 -> 4
- net /INT3: track 0.00 -> 119.4 mm, vias 0 -> 1
- net /EN3: track 0.00 -> 100.1 mm, vias 0 -> 4
- net /INT2: track 0.00 -> 92.3 mm, vias 0 -> 1
- net /INT1: track 143.7 -> 65.8 mm, vias 0 -> 1
- net /EN2: track 0.00 -> 72.9 mm, vias 0 -> 4
- net /Isolated Atlas OEM Module/SDA_3V3: track 67.5 -> 0.00 mm
- net /Isolated Atlas OEM Module/SCL_3V3: track 66.2 -> 0.00 mm
- net /Isolated Atlas OEM Module/ISO_3V3: track 53.3 -> 0.00 mm, vias 24 -> 0
- net Net-(Q4-S): track 70.7 -> 17.7 mm
- net /SCL_SOFT: track 0.00 -> 50.4 mm, vias 0 -> 1
- net /EN1: track 14.1 -> 63.9 mm
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- added copper zone on In1.Cu, net +5V
- added copper zone on In2.Cu, net /ISO1_3V3
- added copper zone on B.Cu, net /ISO1_GND
- added copper zone on F.Cu, net /ISO1_GND
- added copper zone on In1.Cu, net /ISO1_GND
- added copper zone on In2.Cu, net /ISO2_3V3
- added copper zone on B.Cu, net /ISO2_GND
- added copper zone on F.Cu, net /ISO2_GND
- added copper zone on In1.Cu, net /ISO2_GND
- added copper zone on In2.Cu, net /ISO3_3V3
- added copper zone on B.Cu, net /ISO3_GND
- added copper zone on F.Cu, net /ISO3_GND
- added copper zone on In1.Cu, net /ISO3_GND
- added copper zone on In2.Cu, net /ISO4_3V3
- added copper zone on B.Cu, net /ISO4_GND
- added copper zone on F.Cu, net /ISO4_GND
- added copper zone on In1.Cu, net /ISO4_GND
- added copper zone on B.Cu, net /Isolated Atlas OEM Module1/REF_1
- added copper zone on F.Cu, net /Isolated Atlas OEM Module1/REF_1
- added copper zone on In1.Cu, net /Isolated Atlas OEM Module1/REF_1
- added copper zone on In2.Cu, net /Isolated Atlas OEM Module1/REF_1
- added copper zone on F.Cu, net /Isolated Atlas OEM Module1/REF_2
- added copper zone on In1.Cu, net /Isolated Atlas OEM Module1/REF_2
- added copper zone on B.Cu, net /Isolated Atlas OEM Module2/REF_1
- added copper zone on F.Cu, net /Isolated Atlas OEM Module2/REF_1
- added copper zone on In1.Cu, net /Isolated Atlas OEM Module2/REF_1
- added copper zone on In2.Cu, net /Isolated Atlas OEM Module2/REF_1
- added copper zone on B.Cu, net /Isolated Atlas OEM Module2/REF_2
- added copper zone on F.Cu, net /Isolated Atlas OEM Module2/REF_2
- added copper zone on In1.Cu, net /Isolated Atlas OEM Module2/REF_2
- added copper zone on In2.Cu, net /Isolated Atlas OEM Module2/REF_2
- added copper zone on B.Cu, net /Isolated Atlas OEM Module3/REF_1
- added copper zone on F.Cu, net /Isolated Atlas OEM Module3/REF_1
- added copper zone on In1.Cu, net /Isolated Atlas OEM Module3/REF_1
- added copper zone on In2.Cu, net /Isolated Atlas OEM Module3/REF_1
- added copper zone on B.Cu, net /Isolated Atlas OEM Module3/REF_2
- added copper zone on F.Cu, net /Isolated Atlas OEM Module3/REF_2
- added copper zone on In1.Cu, net /Isolated Atlas OEM Module3/REF_2
- added copper zone on In2.Cu, net /Isolated Atlas OEM Module3/REF_2
- added copper zone on B.Cu, net /Isolated Atlas OEM Module4/REF_1
- added copper zone on F.Cu, net /Isolated Atlas OEM Module4/REF_1
- added copper zone on In1.Cu, net /Isolated Atlas OEM Module4/REF_1
- added copper zone on In2.Cu, net /Isolated Atlas OEM Module4/REF_1
- added copper zone on B.Cu, net /Isolated Atlas OEM Module4/REF_2
- added copper zone on F.Cu, net /Isolated Atlas OEM Module4/REF_2
- added copper zone on In1.Cu, net /Isolated Atlas OEM Module4/REF_2
- added copper zone on In2.Cu, net /Isolated Atlas OEM Module4/REF_2
- removed copper zone on In2.Cu, net +12V
- removed copper zone on In2.Cu, net +5V
- removed copper zone on In1.Cu, net /Isolated Atlas OEM Module/ADM3260 I2C Isolator1/AVCC
- removed copper zone on In2.Cu, net /Isolated Atlas OEM Module/ISO_3V3
- removed copper zone on B.Cu, net /Isolated Atlas OEM Module/ISO_GND
- removed copper zone on F.Cu, net /Isolated Atlas OEM Module/ISO_GND
- removed copper zone on In1.Cu, net /Isolated Atlas OEM Module/ISO_GND
- removed copper zone on F.Cu, net /Isolated Atlas OEM Module/PROBE_IN3
- removed copper zone on In1.Cu, net /Isolated Atlas OEM Module/PROBE_IN3
- removed copper zone on B.Cu, net /Isolated Atlas OEM Module/REF_1
- removed copper zone on In2.Cu, net /Isolated Atlas OEM Module/REF_1
- removed copper zone on F.Cu, net /Isolated Atlas OEM Module1/SIG_1
- removed copper zone on In1.Cu, net /Isolated Atlas OEM Module1/SIG_1
- removed copper zone on In1.Cu, net GND
- removed copper zone on In1.Cu, net GNDPWR
Other:
- board text added: "BREAD Slice Atlas.Sci. OEM Multi. SLC_AOEM R3 05-2025"
- board text added: "REG."
- board text added: "SPLIT"
- board text added: "War! The Republic is crumbling under attacks by the ruthless Sith Lord, Count Dooku. There are heroes on both sides. Evil is everywhere. In a stunning move, the fiendish droid leader, General Grievous, has swept into the Republic capital and kidnapped Chancellor Palpatine, leader of the Galactic Senate. As the Separatist Droid Army attempts to flee the besieged capital with their valuable hostage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"
- board text removed: "BREAD Slice 4-layer-XL SLC_TEMP-4LXL R3 04-2025"
- board text removed: "L1 (Top): - Template digital components (Nano, RGB LED) and I²C signals - use minimal ground pours. L2 (Inner 1): - Solid ground plane - split into an upper {dblquote}gndpwr{dblquote} zone (handling 12V returns) and a lower digital ground zone, connected only at the regulator - these can be resized to accommadate additional planes - i.e. decreasing 12V/GNDPWR planes to connector edge and creating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"
