File: hardware-new/adm3260.kicad_sch (KiCad schematic)
At the start: 18 parts, among them Q1 BSS84, Q2 BS170, Q3 BSS84, U3 ADM3260ARSZ

Commit message: finalized pcb
Parts:
- renumbered U3 to U2
Connections:
- net AVCC: no longer R1.1, R2.1
- net VCC: now also R1.1, R2.1
Other:
- moved on the sheet: Q1, Q2, Q3
