File: hardware-new/iso_atlas_oem.kicad_sch (KiCad schematic)
At the start: 4 parts, among them J2 Conn_Coaxial, J3 Conn_Coaxial, U2 Atlas Scientific OEM

Commit message: finalized pcb
Parts:
- renumbered JP9 to JP3, U2 to U3
Connections:
- net REF_1: now also JP3.3 (B); no longer JP3.2 (C)
- net PROBE_IN1 renamed SIG_1
- net PROBE_IN2 renamed PRB_IN2_SEL
- net PRB_IN2_SEL: now also JP3.2 (C); no longer JP3.1 (A)
- net PROBE_IN3 renamed SIG_2
- net SIG_2: now also JP3.1 (A); no longer JP3.3 (B)
- net PROBE_IN4 renamed REF_2
Other:
- removed sheet ADM3260 I2C Isolator1
- note removed: "I2C Isolation"
- moved on the sheet: J2, J3, JP3, U3
