File: hardware/adm3260.kicad_sch (KiCad schematic)
At the start: 18 parts, among them Q1 BSS84, Q2 BS170, Q3 BSS84, U2 ADM3260ARSZ

Commit message: chores: clean up warnings and part references
Parts:
- U2: footprint kml-custom:RS_20_ADI-L -> KMLib_IC_SMD:RS_20_ADI; symbol kml-custom:ADM3260ARSZ -> KMLib_IC_Digital:ADM3260ARSZ_Digital_Isolator
Changed lines of the file:
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@@
 	)
 	(symbol
-		(lib_id "kml-custom:ADM3260ARSZ")
+		(lib_id "KMLib_IC_Digital:ADM3260ARSZ_Digital_Isolator")
 		(at 110.49 82.55 0)
 		(unit 1)
@@
 			)
 		)
-		(property "Footprint" "kml-custom:RS_20_ADI-L"
+		(property "Footprint" "KMLib_IC_SMD:RS_20_ADI"
 			(at 110.49 82.55 0)
 			(hide yes)
