File: hardware/BREAD_Slice.kicad_pcb (KiCad board)
At the start: 4 copper layers, 100.1 x 144.9 mm, 107 parts, among them J1 Conn_01x10_Female, J2 Conn_Coaxial, J3 Conn_Coaxial, J4 Conn_Coaxial, J5 Conn_Coaxial, J6 Conn_Coaxial, J7 Conn_Coaxial, J8 Conn_Coaxial, J9 Conn_Coaxial, Q1 BSS84, Q10 BSS84, Q11 BS170, Q12 BSS84, Q2 BS170, Q3 BSS84, Q4 BSS84, Q5 BS170, Q6 BSS84, Q7 BSS84, Q8 BS170, Q9 BSS84, U1 AP63205, U2 ADM3260ARSZ, U3 Atlas Scientific OEM, U4 ADM3260ARSZ, U5 Atlas Scientific OEM, U6 ADM3260ARSZ, U7 Atlas Scientific OEM, U8 ADM3260ARSZ, U9 Atlas Scientific OEM

Commit message: fix(hw): re-point stale library nicknames
These parts exist in KiCad-Master-Lib; the boards referenced libraries that no
longer exist (kml-custom, KML-Custom, and SparkFun libraries that never
contained the part) or names the library has since changed.

KiCad embeds footprint geometry in the .kicad_pcb, so the boards rendered and
fabricated correctly and the rot stayed invisible -- it only surfaces on
update-from-library, or when a generator tries to resolve a nickname.

Nickname/name only. No geometry is changed:

  KMLib_Mounting:Thermal Pad -> KMLib_Mounting:Thermal_Pad
  SparkFun-LED:WS2812-5050-4PIN -> KMLib_IC_SMD:WS2812-5050-4PIN
  kml-custom:Atlas_OEM -> KMLib_Boards_Modules:Atlas_OEM
  kml-custom:FAST-Logo-XXXLarge -> KMLib_Aesthetic:FAST-Logo-XXXLarge
  kml-custom:RS_20_ADI-L -> KMLib_IC_SMD:RS_20_ADI-L
  kml-custom:Thermal Pad -> KMLib_Mounting:Thermal_Pad

Only references that failed to resolve were touched. Generic parts (<=4 pins)
and KiCad *-rescue libraries are deliberately excluded: fingerprint matching
cannot distinguish a 2-pin resistor from a 2-pin capacitor, so those are being
done by hand.
Parts:
- D1: footprint SparkFun-LED:WS2812-5050-4PIN -> KMLib_IC_SMD:WS2812-5050-4PIN
- G***: footprint kml-custom:FAST-Logo-XXXLarge -> KMLib_Aesthetic:FAST-Logo-XXXLarge
- HS1: footprint kml-custom:Thermal Pad -> KMLib_Mounting:Thermal_Pad
- U2, U4, U6, U8: footprint kml-custom:RS_20_ADI-L -> KMLib_IC_SMD:RS_20_ADI-L
- U3, U5, U7, U9: footprint kml-custom:Atlas_OEM -> KMLib_Boards_Modules:Atlas_OEM
Changed lines of the file:
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@@
 		)
 	)
-	(footprint "kml-custom:RS_20_ADI-L"
+	(footprint "KMLib_IC_SMD:RS_20_ADI-L"
 		(layer "F.Cu")
 		(at 122.388799 92.261991)
@@
 		)
 	)
-	(footprint "kml-custom:RS_20_ADI-L"
+	(footprint "KMLib_IC_SMD:RS_20_ADI-L"
 		(layer "F.Cu")
 		(at 122.348985 122.261432)
@@
 		)
 	)
-	(footprint "kml-custom:Atlas_OEM"
+	(footprint "KMLib_Boards_Modules:Atlas_OEM"
 		(layer "F.Cu")
 		(at 146.660124 69.186598 90)
@@
 		)
 	)
-	(footprint "SparkFun-LED:WS2812-5050-4PIN"
+	(footprint "KMLib_IC_SMD:WS2812-5050-4PIN"
 		(locked yes)
 		(layer "F.Cu")
@@
 		)
 	)
-	(footprint "kml-custom:Atlas_OEM"
+	(footprint "KMLib_Boards_Modules:Atlas_OEM"
 		(layer "F.Cu")
 		(at 146.638722 159.33645 90)
@@
 		)
 	)
-	(footprint "kml-custom:FAST-Logo-XXXLarge"
+	(footprint "KMLib_Aesthetic:FAST-Logo-XXXLarge"
 		(layer "F.Cu")
 		(at 85.87 72.61)
@@
 		)
 	)
-	(footprint "kml-custom:Atlas_OEM"
+	(footprint "KMLib_Boards_Modules:Atlas_OEM"
 		(layer "F.Cu")
 		(at 146.647258 98.66645 90)
@@
 		)
 	)
-	(footprint "kml-custom:Thermal Pad"
+	(footprint "KMLib_Mounting:Thermal_Pad"
 		(layer "F.Cu")
 		(at 66.774465 162.653932)
@@
 		)
 	)
-	(footprint "kml-custom:RS_20_ADI-L"
+	(footprint "KMLib_IC_SMD:RS_20_ADI-L"
 		(layer "F.Cu")
 		(at 122.380263 152.929746)
@@
 		)
 	)
-	(footprint "kml-custom:Atlas_OEM"
+	(footprint "KMLib_Boards_Modules:Atlas_OEM"
 		(layer "F.Cu")
 		(at 146.608722 128.666686 90)
@@
 		)
 	)
-	(footprint "kml-custom:RS_20_ADI-L"
+	(footprint "KMLib_IC_SMD:RS_20_ADI-L"
 		(layer "F.Cu")
 		(at 122.395387 62.776344)
